Commit message: URDF update complete. Implemented class based actuator configuration. Flipped joint actuation torque signage for motors inverted on model to ensure correct hardware outputs.

File: source/BDXR/data/Robots/BDXR/URDF.urdf (robot description, URDF)
Before this commit: robot URDF, 77 links, 76 joints
Links:
- removed link Front_Grill
- removed link Head_Rear_Cover
- added link Left_Ear_Holder, mass 0.039089198133902825; collision mesh filename=meshes/Left_Ear_Holder.stl scale=0.001 0.001 0.001; visual mesh filename=meshes/Left_Ear_Holder.stl scale=0.001 0.001 0.001
- added link Left_Ear_Motor, mass 0.21407639017138763; collision mesh filename=meshes/Left_Ear_Motor.stl scale=0.001 0.001 0.001; visual mesh filename=meshes/Left_Ear_Motor.stl scale=0.001 0.001 0.001
- added link Orin_Nano_Case, mass 0.5; collision mesh filename=meshes/Orin_Nano_Case.stl scale=0.001 0.001 0.001; visual mesh filename=meshes/Orin_Nano_Case.stl scale=0.001 0.001 0.001
- added link Rear_Head_Cover, mass 0.3; collision mesh filename=meshes/Rear_Head_Cover.stl scale=0.001 0.001 0.001; visual mesh filename=meshes/Rear_Head_Cover.stl scale=0.001 0.001 0.001
- added link Right_Ear_Holder, mass 0.039089198133902665; collision mesh filename=meshes/Right_Ear_Holder.stl scale=0.001 0.001 0.001; visual mesh filename=meshes/Right_Ear_Holder.stl scale=0.001 0.001 0.001
- added link Right_Ear_Motor, mass 0.21407640350583973; collision mesh filename=meshes/Right_Ear_Motor.stl scale=0.001 0.001 0.001; visual mesh filename=meshes/Right_Ear_Motor.stl scale=0.001 0.001 0.001
- link Back_Support: mass 0.1 -> 0.19818519083453695; geometry collision mesh filename=meshes/Back_Support.stl scale=0.001 0.001 0.001; visual mesh filename=meshes/Back_Support.stl scale=0.001 0.001 0.001
- link Base_Top_Clamp: mass 0.044 -> 0.04628859676338927; geometry collision mesh filename=meshes/Base_Top_Clamp.stl scale=0.001 0.001 0.001; visual mesh filename=meshes/Base_Top_Clamp.stl scale=0.001 0.001 0.001
- link Battery: mass 1.25 -> 1.073094288437329; geometry collision mesh filename=meshes/Battery.stl scale=0.001 0.001 0.001; visual mesh filename=meshes/Battery.stl scale=0.001 0.001 0.001
- link Battery_Holder: mass 0.18 -> 0.16209189271424795; geometry collision mesh filename=meshes/Battery_Holder.stl scale=0.001 0.001 0.001; visual mesh filename=meshes/Battery_Holder.stl scale=0.001 0.001 0.001
- link Bottom_Cover: geometry collision mesh filename=meshes/Bottom_Cover.stl scale=0.001 0.001 0.001; visual mesh filename=meshes/Bottom_Cover.stl scale=0.001 0.001 0.001
- link Camera_Mount: mass 0.04 -> 0.032111017172493185; geometry collision mesh filename=meshes/Camera_Mount.stl scale=0.001 0.001 0.001; visual mesh filename=meshes/Camera_Mount.stl scale=0.001 0.001 0.001
- link Face: mass 0.1 -> 0.036547681364044626; geometry collision mesh filename=meshes/Face.stl scale=0.001 0.001 0.001; visual mesh filename=meshes/Face.stl scale=0.001 0.001 0.001
- link Front_Cover: mass 0.2 -> 0.319189974357708; geometry collision mesh filename=meshes/Front_Cover.stl scale=0.001 0.001 0.001; visual mesh filename=meshes/Front_Cover.stl scale=0.001 0.001 0.001
- link Front_Support: mass 0.15 -> 0.18424409661297098; geometry collision mesh filename=meshes/Front_Support.stl scale=0.001 0.001 0.001; visual mesh filename=meshes/Front_Support.stl scale=0.001 0.001 0.001
- link Head_Base_Plate: mass 0.24 -> 0.24167712099257307; geometry collision mesh filename=meshes/Head_Base_Plate.stl scale=0.001 0.001 0.001; visual mesh filename=meshes/Head_Base_Plate.stl scale=0.001 0.001 0.001
- link Head_Pitch_Motor: mass 0.242 -> 0.21407641363122526; geometry collision mesh filename=meshes/Head_Pitch_Motor.stl scale=0.001 0.001 0.001; visual mesh filename=meshes/Head_Pitch_Motor.stl scale=0.001 0.001 0.001
- link Head_Pitch_Motor_Support: mass 0.08 -> 0.04464301349288608; geometry collision mesh filename=meshes/Head_Pitch_Motor_Support.stl scale=0.001 0.001 0.001; visual mesh filename=meshes/Head_Pitch_Motor_Support.stl scale=0.001 0.001 0.001
- link Head_Roll_Connector: mass 0.05 -> 0.02623495760996857; geometry collision mesh filename=meshes/Head_Roll_Connector.stl scale=0.001 0.001 0.001; visual mesh filename=meshes/Head_Roll_Connector.stl scale=0.001 0.001 0.001
- link Head_Roll_Motor: mass 0.242 -> 0.21407532118731826; geometry collision mesh filename=meshes/Head_Roll_Motor.stl scale=0.001 0.001 0.001; visual mesh filename=meshes/Head_Roll_Motor.stl scale=0.001 0.001 0.001
- link Head_Roll_Motor_Mount: mass 0.08 -> 0.06069341482294389; geometry collision mesh filename=meshes/Head_Roll_Motor_Mount.stl scale=0.001 0.001 0.001; visual mesh filename=meshes/Head_Roll_Motor_Mount.stl scale=0.001 0.001 0.001
- link Head_Yaw_Motor: mass 0.242 -> 0.214075321187319; geometry collision mesh filename=meshes/Head_Yaw_Motor.stl scale=0.001 0.001 0.001; visual mesh filename=meshes/Head_Yaw_Motor.stl scale=0.001 0.001 0.001
- link Left_Ankle_Cover: mass 0.01 -> 0.014202085744813586; geometry collision mesh filename=meshes/Left_Ankle_Cover.stl scale=0.001 0.001 0.001; visual mesh filename=meshes/Left_Ankle_Cover.stl scale=0.001 0.001 0.001
- link Left_Ankle_Motor: mass 0.405 -> 0.43362988206706554; geometry collision mesh filename=meshes/Left_Ankle_Motor.stl scale=0.001 0.001 0.001; visual mesh filename=meshes/Left_Ankle_Motor.stl scale=0.001 0.001 0.001
- link Left_Cable_Support: mass 0.08 -> 0.05527465492344571; geometry collision mesh filename=meshes/Left_Cable_Support.stl scale=0.001 0.001 0.001; visual mesh filename=meshes/Left_Cable_Support.stl scale=0.001 0.001 0.001
- link Left_Ear: mass 0.01 -> 0.0173058023178019; geometry collision mesh filename=meshes/Left_Ear.stl scale=0.001 0.001 0.001; visual mesh filename=meshes/Left_Ear.stl scale=0.001 0.001 0.001
- link Left_Eye: mass 0.02 -> 0.010759900541269532; geometry collision mesh filename=meshes/Left_Eye.stl scale=0.001 0.001 0.001; visual mesh filename=meshes/Left_Eye.stl scale=0.001 0.001 0.001
- link Left_Foot: mass 0.22 -> 0.253738845261166; geometry collision mesh filename=meshes/Left_Foot.stl scale=0.001 0.001 0.001; visual mesh filename=meshes/Left_Foot.stl scale=0.001 0.001 0.001
- link Left_Foot_Cover: mass 0.02 -> 0.03752369551950594; geometry collision mesh filename=meshes/Left_Foot_Cover.stl scale=0.001 0.001 0.001; visual mesh filename=meshes/Left_Foot_Cover.stl scale=0.001 0.001 0.001
- link Left_Foot_Pad: mass 0.08 -> 0.11120287867405936; geometry collision mesh filename=meshes/Left_Foot_Pad.stl scale=0.001 0.001 0.001; visual mesh filename=meshes/Left_Foot_Pad.stl scale=0.001 0.001 0.001
- link Left_Front_Cover: mass 0.1 -> 0.05247574794931451; geometry collision mesh filename=meshes/Left_Front_Cover.stl scale=0.001 0.001 0.001; visual mesh filename=meshes/Left_Front_Cover.stl scale=0.001 0.001 0.001
- link Left_Head_Support: mass 0.04 -> 0.020436827848287157; geometry collision mesh filename=meshes/Left_Head_Support.stl scale=0.001 0.001 0.001; visual mesh filename=meshes/Left_Head_Support.stl scale=0.001 0.001 0.001
- link Left_Hip_Bottom_Holder: mass 0.075 -> 0.06006501163237421; geometry collision mesh filename=meshes/Left_Hip_Bottom_Holder.stl scale=0.001 0.001 0.001; visual mesh filename=meshes/Left_Hip_Bottom_Holder.stl scale=0.001 0.001 0.001
- link Left_Hip_Pitch_Motor: mass 0.920 -> 0.9104515289190356; geometry collision mesh filename=meshes/Left_Hip_Pitch_Motor.stl scale=0.001 0.001 0.001; visual mesh filename=meshes/Left_Hip_Pitch_Motor.stl scale=0.001 0.001 0.001
- link Left_Hip_Roll_Connector: mass 0.1 -> 0.09814593711615145; geometry collision mesh filename=meshes/Left_Hip_Roll_Connector.stl scale=0.001 0.001 0.001; visual mesh filename=meshes/Left_Hip_Roll_Connector.stl scale=0.001 0.001 0.001
- link Left_Hip_Roll_Motor: mass 0.920 -> 0.9069870657157226; geometry collision mesh filename=meshes/Left_Hip_Roll_Motor.stl scale=0.001 0.001 0.001; visual mesh filename=meshes/Left_Hip_Roll_Motor.stl scale=0.001 0.001 0.001
- link Left_Hip_Top_Holder: mass 0.08 -> 0.08211265972988092; geometry collision mesh filename=meshes/Left_Hip_Top_Holder.stl scale=0.001 0.001 0.001; visual mesh filename=meshes/Left_Hip_Top_Holder.stl scale=0.001 0.001 0.001
- link Left_Hip_Yaw_Motor: mass 0.920 -> 0.9104438184229293; geometry collision mesh filename=meshes/Left_Hip_Yaw_Motor.stl scale=0.001 0.001 0.001; visual mesh filename=meshes/Left_Hip_Yaw_Motor.stl scale=0.001 0.001 0.001
- link Left_Hip_Yaw_Support: mass 0.08 -> 0.10788076345385224; geometry collision mesh filename=meshes/Left_Hip_Yaw_Support.stl scale=0.001 0.001 0.001; visual mesh filename=meshes/Left_Hip_Yaw_Support.stl scale=0.001 0.001 0.001
- link Left_Holder: mass 0.08 -> 0.03609216827781493; geometry collision mesh filename=meshes/Left_Holder.stl scale=0.001 0.001 0.001; visual mesh filename=meshes/Left_Holder.stl scale=0.001 0.001 0.001
- link Left_Knee_Motor: mass 0.920 -> 0.9104515217073631; geometry collision mesh filename=meshes/Left_Knee_Motor.stl scale=0.001 0.001 0.001; visual mesh filename=meshes/Left_Knee_Motor.stl scale=0.001 0.001 0.001
- link Left_Lower_Leg: mass 0.33 -> 0.3868529143335189; geometry collision mesh filename=meshes/Left_Lower_Leg.stl scale=0.001 0.001 0.001; visual mesh filename=meshes/Left_Lower_Leg.stl scale=0.001 0.001 0.001
- link Left_Lower_Leg_Cover: mass 0.057 -> 0.09180221523312034; geometry collision mesh filename=meshes/Left_Lower_Leg_Cover.stl scale=0.001 0.001 0.001; visual mesh filename=meshes/Left_Lower_Leg_Cover.stl scale=0.001 0.001 0.001
- link Left_Top_Cover: mass 0.03 -> 0.02926093594411759; geometry collision mesh filename=meshes/Left_Top_Cover.stl scale=0.001 0.001 0.001; visual mesh filename=meshes/Left_Top_Cover.stl scale=0.001 0.001 0.001
- link Left_Upper_Leg: mass 0.5 -> 0.5655536567558276; geometry collision mesh filename=meshes/Left_Upper_Leg.stl scale=0.001 0.001 0.001; visual mesh filename=meshes/Left_Upper_Leg.stl scale=0.001 0.001 0.001
- link Left_Upper_Leg_Cover: mass 0.075 -> 0.0636117280594398; geometry collision mesh filename=meshes/Left_Upper_Leg_Cover.stl scale=0.001 0.001 0.001; visual mesh filename=meshes/Left_Upper_Leg_Cover.stl scale=0.001 0.001 0.001
- link Left_Upper_Leg_Detail: mass 0.01 -> 0.004967595085878627; geometry collision mesh filename=meshes/Left_Upper_Leg_Detail.stl scale=0.001 0.001 0.001; visual mesh filename=meshes/Left_Upper_Leg_Detail.stl scale=0.001 0.001 0.001
- link Neck: geometry collision mesh filename=meshes/Neck.stl scale=0.001 0.001 0.001; visual mesh filename=meshes/Neck.stl scale=0.001 0.001 0.001
- link Neck_Motor: mass 0.405 -> 0.42940231867124456; geometry collision mesh filename=meshes/Neck_Motor.stl scale=0.001 0.001 0.001; visual mesh filename=meshes/Neck_Motor.stl scale=0.001 0.001 0.001
- link Rear_Antenna_Box: mass 0.1 -> 0.04117094798631419; geometry collision mesh filename=meshes/Rear_Antenna_Box.stl scale=0.001 0.001 0.001; visual mesh filename=meshes/Rear_Antenna_Box.stl scale=0.001 0.001 0.001
- link Rear_Cover: mass 0.15 -> 0.31819716922538754; geometry collision mesh filename=meshes/Rear_Cover.stl scale=0.001 0.001 0.001; visual mesh filename=meshes/Rear_Cover.stl scale=0.001 0.001 0.001
- link Rear_Head_Plate: mass 0.05 -> 0.014787579197992883; geometry collision mesh filename=meshes/Rear_Head_Plate.stl scale=0.001 0.001 0.001; visual mesh filename=meshes/Rear_Head_Plate.stl scale=0.001 0.001 0.001
- link Right_Ankle_Cover: mass 0.01 -> 0.014202085744813589; geometry collision mesh filename=meshes/Right_Ankle_Cover.stl scale=0.001 0.001 0.001; visual mesh filename=meshes/Right_Ankle_Cover.stl scale=0.001 0.001 0.001
- link Right_Ankle_Motor: mass 0.405 -> 0.43363012395690076; geometry collision mesh filename=meshes/Right_Ankle_Motor.stl scale=0.001 0.001 0.001; visual mesh filename=meshes/Right_Ankle_Motor.stl scale=0.001 0.001 0.001
- link Right_Cable_Support: mass 0.08 -> 0.055274654923445694; geometry collision mesh filename=meshes/Right_Cable_Support.stl scale=0.001 0.001 0.001; visual mesh filename=meshes/Right_Cable_Support.stl scale=0.001 0.001 0.001
- link Right_Ear: mass 0.01 -> 0.017330282593122717; geometry collision mesh filename=meshes/Right_Ear.stl scale=0.001 0.001 0.001; visual mesh filename=meshes/Right_Ear.stl scale=0.001 0.001 0.001
- link Right_Eye: mass 0.02 -> 0.011103671152706012; geometry collision mesh filename=meshes/Right_Eye.stl scale=0.001 0.001 0.001; visual mesh filename=meshes/Right_Eye.stl scale=0.001 0.001 0.001
- link Right_Foot: mass 0.22 -> 0.25373884525351503; geometry collision mesh filename=meshes/Right_Foot.stl scale=0.001 0.001 0.001; visual mesh filename=meshes/Right_Foot.stl scale=0.001 0.001 0.001
- link Right_Foot_Cover: mass 0.02 -> 0.037524104890090594; geometry collision mesh filename=meshes/Right_Foot_Cover.stl scale=0.001 0.001 0.001; visual mesh filename=meshes/Right_Foot_Cover.stl scale=0.001 0.001 0.001
- link Right_Foot_Pad: mass 0.08 -> 0.11120287867405933; geometry collision mesh filename=meshes/Right_Foot_Pad.stl scale=0.001 0.001 0.001; visual mesh filename=meshes/Right_Foot_Pad.stl scale=0.001 0.001 0.001
- link Right_Front_Cover: mass 0.1 -> 0.053605686719820106; geometry collision mesh filename=meshes/Right_Front_Cover.stl scale=0.001 0.001 0.001; visual mesh filename=meshes/Right_Front_Cover.stl scale=0.001 0.001 0.001
- link Right_Head_Support: mass 0.04 -> 0.020436827877729553; geometry collision mesh filename=meshes/Right_Head_Support.stl scale=0.001 0.001 0.001; visual mesh filename=meshes/Right_Head_Support.stl scale=0.001 0.001 0.001
- link Right_Hip_Bottom_Holder: mass 0.075 -> 0.060065011632374196; geometry collision mesh filename=meshes/Right_Hip_Bottom_Holder.stl scale=0.001 0.001 0.001; visual mesh filename=meshes/Right_Hip_Bottom_Holder.stl scale=0.001 0.001 0.001
- link Right_Hip_Pitch_Motor: mass 0.920 -> 0.9104438192734086; geometry collision mesh filename=meshes/Right_Hip_Pitch_Motor.stl scale=0.001 0.001 0.001; visual mesh filename=meshes/Right_Hip_Pitch_Motor.stl scale=0.001 0.001 0.001
- link Right_Hip_Roll_Connector: mass 0.1 -> 0.09814591729138275; geometry collision mesh filename=meshes/Right_Hip_Roll_Connector.stl scale=0.001 0.001 0.001; visual mesh filename=meshes/Right_Hip_Roll_Connector.stl scale=0.001 0.001 0.001
- link Right_Hip_Roll_Motor: mass 0.920 -> 0.9069872059005614; geometry collision mesh filename=meshes/Right_Hip_Roll_Motor.stl scale=0.001 0.001 0.001; visual mesh filename=meshes/Right_Hip_Roll_Motor.stl scale=0.001 0.001 0.001
- link Right_Hip_Top_Holder: mass 0.08 -> 0.08211265972988097; geometry collision mesh filename=meshes/Right_Hip_Top_Holder.stl scale=0.001 0.001 0.001; visual mesh filename=meshes/Right_Hip_Top_Holder.stl scale=0.001 0.001 0.001
- link Right_Hip_Yaw_Motor: mass 0.920 -> 0.9104438183269751; geometry collision mesh filename=meshes/Right_Hip_Yaw_Motor.stl scale=0.001 0.001 0.001; visual mesh filename=meshes/Right_Hip_Yaw_Motor.stl scale=0.001 0.001 0.001
- link Right_Hip_Yaw_Support: mass 0.08 -> 0.11096680121360432; geometry collision mesh filename=meshes/Right_Hip_Yaw_Support.stl scale=0.001 0.001 0.001; visual mesh filename=meshes/Right_Hip_Yaw_Support.stl scale=0.001 0.001 0.001
- link Right_Holder: mass 0.08 -> 0.03611281660144922; geometry collision mesh filename=meshes/Right_Holder.stl scale=0.001 0.001 0.001; visual mesh filename=meshes/Right_Holder.stl scale=0.001 0.001 0.001
- link Right_Knee_Motor: mass 0.920 -> 0.9104438184284508; geometry collision mesh filename=meshes/Right_Knee_Motor.stl scale=0.001 0.001 0.001; visual mesh filename=meshes/Right_Knee_Motor.stl scale=0.001 0.001 0.001
- link Right_Lower_Leg: mass 0.33 -> 0.38685291363183144; geometry collision mesh filename=meshes/Right_Lower_Leg.stl scale=0.001 0.001 0.001; visual mesh filename=meshes/Right_Lower_Leg.stl scale=0.001 0.001 0.001
- link Right_Lower_Leg_Cover: mass 0.057 -> 0.04937375027674599; geometry collision mesh filename=meshes/Right_Lower_Leg_Cover.stl scale=0.001 0.001 0.001; visual mesh filename=meshes/Right_Lower_Leg_Cover.stl scale=0.001 0.001 0.001
- link Right_Top_Cover: mass 0.03 -> 0.029260935944117595; geometry collision mesh filename=meshes/Right_Top_Cover.stl scale=0.001 0.001 0.001; visual mesh filename=meshes/Right_Top_Cover.stl scale=0.001 0.001 0.001
- link Right_Upper_Leg: mass 0.5 -> 0.5655879310958503; geometry collision mesh filename=meshes/Right_Upper_Leg.stl scale=0.001 0.001 0.001; visual mesh filename=meshes/Right_Upper_Leg.stl scale=0.001 0.001 0.001
- link Right_Upper_Leg_Cover: mass 0.075 -> 0.0636117280607867; geometry collision mesh filename=meshes/Right_Upper_Leg_Cover.stl scale=0.001 0.001 0.001; visual mesh filename=meshes/Right_Upper_Leg_Cover.stl scale=0.001 0.001 0.001
- link Right_Upper_Leg_Detail: mass 0.01 -> 0.004967595005976366; geometry collision mesh filename=meshes/Right_Upper_Leg_Detail.stl scale=0.001 0.001 0.001; visual mesh filename=meshes/Right_Upper_Leg_Detail.stl scale=0.001 0.001 0.001
- link Top_Base_Frame: mass 0.15 -> 0.1195092727509324; geometry collision mesh filename=meshes/Top_Base_Frame.stl scale=0.001 0.001 0.001; visual mesh filename=meshes/Top_Base_Frame.stl scale=0.001 0.001 0.001
- link base_link: mass 1 -> 1.1588690647920126; geometry collision mesh filename=meshes/base_link.stl scale=0.001 0.001 0.001; visual mesh filename=meshes/base_link.stl scale=0.001 0.001 0.001
- link imu: mass 0.05 -> 0.1; geometry collision mesh filename=meshes/imu.stl scale=0.001 0.001 0.001; visual mesh filename=meshes/imu.stl scale=0.001 0.001 0.001
- link imu_mount: mass 0.03 -> 0.05; geometry collision mesh filename=meshes/imu_mount.stl scale=0.001 0.001 0.001; visual mesh filename=meshes/imu_mount.stl scale=0.001 0.001 0.001
Joints:
- removed joint Rigid 37
- removed joint Rigid 38
- removed joint Rigid 39
- removed joint Rigid 40
- removed joint Rigid 58
- added joint Rigid 80: type fixed, parent Front_Support, child Orin_Nano_Case, origin xyz=0.01 -0.02 0.0 rpy=0 0 0
- added joint Rigid 81: type fixed, parent Head_Base_Plate, child Right_Ear_Holder, origin xyz=-0.142593 -0.04359 0.0 rpy=0 0 0
- added joint Rigid 82: type fixed, parent Right_Ear_Holder, child Right_Ear_Motor, origin xyz=-0.021543 0.004139 0.045321 rpy=0 0 0
- added joint Rigid 83: type fixed, parent Right_Ear_Motor, child Right_Ear, origin xyz=0.000669 0.0 -0.019584 rpy=0 0 0
- added joint Rigid 84: type fixed, parent Head_Base_Plate, child Left_Ear_Holder, origin xyz=-0.142593 0.067109 0.0 rpy=0 0 0
- added joint Rigid 85: type fixed, parent Left_Ear_Holder, child Left_Ear_Motor, origin xyz=-0.01245 0.024261 0.032311 rpy=0 0 0
- added joint Rigid 86: type fixed, parent Left_Ear_Motor, child Left_Ear, origin xyz=-0.012545 0.0 0.004702 rpy=0 0 0
- added joint Rigid 87: type fixed, parent Left_Head_Support, child Rear_Head_Cover, origin xyz=-0.008598 -0.001727 0.010956 rpy=0 0 0
- added joint Rigid 88: type fixed, parent Rear_Head_Cover, child Rear_Head_Plate, origin xyz=-0.174901 -0.091107 -0.001821 rpy=0 0 0
- joint Head_Pitch: axis (none) -> 0.0 1.0 0.0; limit (none) -> lower=-1.0471975511965976 upper=0.5235987755982988 effort=6.0 velocity=45.0; type fixed -> revolute
- joint Head_Roll: axis (none) -> -1.0 0.0 0.0; limit (none) -> lower=-0.5235987755982988 upper=0.5235987755982988 effort=6.0 velocity=45.0; type fixed -> revolute
- joint Head_Yaw: axis (none) -> 0.0 0.0 -1.0; limit (none) -> lower=-0.8726646259971648 upper=0.8726646259971648 effort=6.0 velocity=45.0; type fixed -> revolute
- joint Left_Ankle: axis 0.0 -1.0 0.0 -> -0.0 -1.0 -0.0
- joint Left_Hip_Pitch: axis 0.0 -1.0 0.0 -> -0.0 1.0 -0.0; limit lower=-1.047 upper=0.698 effort=60.0 velocity=20.0 -> lower=-0.6981317007977318 upper=1.0471975511965976 effort=60.0 velocity=20.0
- joint Left_Hip_Roll: axis -1.0 0.0 0.0 -> 1.0 0.0 -0.0; limit lower=-0.2618 upper=0.349 effort=60.0 velocity=20.0 -> lower=-0.3490658503988659 upper=0.2617993877991494 effort=60.0 velocity=20.0
- joint Left_Knee: axis 0.0 1.0 0.0 -> 0.0 -1.0 0.0; limit lower=-0.9599 upper=1.309 effort=60.0 velocity=20.0 -> lower=-1.3089969389957472 upper=0.9599310885968813 effort=60.0 velocity=20.0; origin xyz=0.045459 -0.0025 0.01829 rpy=0 0 0 -> xyz=0.045459 -0.0025 0.018291 rpy=0 0 0
- joint Neck_Pitch: axis (none) -> 0.0 1.0 -0.0; limit (none) -> lower=-0.3490658503988659 upper=0.8726646259971648 effort=17.0 velocity=43.0; type fixed -> revolute
- joint Right_Ankle: axis 0.0 1.0 0.0 -> 0.0 -1.0 0.0; limit lower=-1.2217 upper=0.785 effort=17.0 velocity=43.0 -> lower=-0.785 upper=1.2217304763960306 effort=17.0 velocity=43.0
- joint Right_Hip_Pitch: axis 0.0 1.0 0.0 -> -0.0 -1.0 -0.0; limit lower=-0.698 upper=1.047 effort=60.0 velocity=20.0 -> lower=-1.0471975511965976 upper=0.6981317007977318 effort=60.0 velocity=20.0
- joint Right_Knee: axis 0.0 -1.0 0.0 -> -0.0 -1.0 -0.0; origin xyz=0.01829 0.0025 -0.045459 rpy=0 0 0 -> xyz=0.01829 0.0025 -0.045458 rpy=0 0 0
- joint Rigid 10: origin xyz=-0.045104 0.01775 0.002892 rpy=0 0 0 -> xyz=0.070648 0.0178 0.088154 rpy=0 0 0
- joint Rigid 11: origin xyz=-0.157 -0.06 0.063636 rpy=0 0 0 -> xyz=-0.041248 -0.05995 0.148898 rpy=0 0 0
- joint Rigid 13: origin xyz=-0.1581 0.090997 0.065042 rpy=0 0 0 -> xyz=-0.042349 0.091047 0.150304 rpy=0 0 0
- joint Rigid 14: origin xyz=-0.148285 0.084346 0.090657 rpy=0 0 0 -> xyz=-0.032533 0.084396 0.175919 rpy=0 0 0
- joint Rigid 16: origin xyz=-0.017969 0.027051 0.074357 rpy=0 0 0 -> xyz=-0.017969 0.027051 0.074557 rpy=0 0 0
- joint Rigid 20: origin xyz=-0.0112 0.01 -0.005406 rpy=0 0 0 -> xyz=0.104552 0.01005 0.079856 rpy=0 0 0
- joint Rigid 23: origin xyz=0.058599 -0.056479 0.0 rpy=0 0 0 -> xyz=0.058598 -0.056479 0.0 rpy=0 0 0
- joint Rigid 24: origin xyz=0.004894 -0.112243 -0.028497 rpy=0 0 0 -> xyz=0.004894 -0.112243 -0.028496 rpy=0 0 0
- joint Rigid 26: origin xyz=0.087134 -0.028034 0.010956 rpy=0 0 0 -> xyz=0.202885 -0.027984 0.096418 rpy=0 0 0
- joint Rigid 27: origin xyz=0.058599 0.109997 0.0 rpy=0 0 0 -> xyz=0.058598 0.109997 0.0 rpy=0 0 0
- joint Rigid 28: origin xyz=-0.1581 -0.090997 0.065042 rpy=0 0 0 -> xyz=-0.042349 -0.090947 0.150304 rpy=0 0 0
- joint Rigid 29: origin xyz=-0.027746 0.157732 0.0 rpy=0 0 0 -> xyz=-0.027747 0.157732 0.0 rpy=0 0 0
- joint Rigid 31: origin xyz=-0.157777 0.0 -0.083128 rpy=0 0 0 -> xyz=-0.042025 5e-05 0.002134 rpy=0 0 0
- joint Rigid 33: origin xyz=-0.024139 -0.0278 0.14533 rpy=0 0 0 -> xyz=0.091613 -0.02775 0.230592 rpy=0 0 0
- joint Rigid 36: origin xyz=0.052962 -0.098148 0.0 rpy=0 0 0 -> xyz=0.052961 -0.098148 0.0 rpy=0 0 0
- joint Rigid 4: origin xyz=-0.148374 0.068751 0.024336 rpy=0 0 0 -> xyz=-0.032622 0.068801 0.109598 rpy=0 0 0
- joint Rigid 49: origin xyz=0.072419 -0.045377 -0.097578 rpy=0 0 0 -> xyz=0.072419 -0.045377 -0.097579 rpy=0 0 0
- joint Rigid 5: origin xyz=-0.148374 -0.068751 0.024336 rpy=0 0 0 -> xyz=-0.032622 -0.068701 0.109598 rpy=0 0 0
- joint Rigid 50: origin xyz=0.009131 -0.00934 -0.124165 rpy=0 0 0 -> xyz=0.009131 -0.00934 -0.124166 rpy=0 0 0
- joint Rigid 52: origin xyz=0.10668 -0.025682 -0.057538 rpy=0 0 0 -> xyz=0.222432 -0.025632 0.027724 rpy=0 0 0
- joint Rigid 54: origin xyz=0.058902 0.0465 -0.075069 rpy=0 0 0 -> xyz=0.058901 0.0465 -0.075069 rpy=0 0 0
- joint Rigid 55: origin xyz=-0.10624 0.0465 -0.111941 rpy=0 0 0 -> xyz=-0.10624 0.0465 -0.11194 rpy=0 0 0
- joint Rigid 56: origin xyz=-0.093612 0.011824 0.044456 rpy=0 0 0 -> xyz=0.022141 0.011874 0.129718 rpy=0 0 0
- joint Rigid 57: origin xyz=0.061778 0.154093 0.101024 rpy=0 0 0 -> xyz=0.177343 0.156643 0.186285 rpy=0 0 0
- joint Rigid 6: origin xyz=0.017134 -0.01645 0.044533 rpy=0 0 0 -> xyz=0.132886 -0.0164 0.129795 rpy=0 0 0
- joint Rigid 68: origin xyz=0.044717 0.00934 -0.09358 rpy=0 0 0 -> xyz=0.044717 0.00934 -0.093581 rpy=0 0 0
- joint Rigid 72: origin xyz=0.058902 -0.0465 -0.075069 rpy=0 0 0 -> xyz=0.058901 -0.0465 -0.075069 rpy=0 0 0
- joint Rigid 73: origin xyz=-0.10624 -0.0465 -0.111941 rpy=0 0 0 -> xyz=-0.10624 -0.0465 -0.11194 rpy=0 0 0
- joint Rigid 74: origin xyz=-0.093612 -0.011824 0.042716 rpy=0 0 0 -> xyz=0.022141 -0.011774 0.127978 rpy=0 0 0
- joint Rigid 75: origin xyz=0.017878 0.045377 -0.162577 rpy=0 0 0 -> xyz=0.017878 0.045377 -0.162578 rpy=0 0 0
- joint Rigid 8: origin xyz=-0.075084 0.063 -0.123908 rpy=0 0 0 -> xyz=0.040668 0.06305 -0.038646 rpy=0 0 0
- joint Rigid 9: origin xyz=-0.045104 -0.01775 0.002892 rpy=0 0 0 -> xyz=0.070648 -0.0177 0.088154 rpy=0 0 0
