Commit message: Built controller, resolved right turn heading bias, turned on self collisions

File: src/BDXR/data/Robots/BDXR/URDF.urdf (robot description, URDF)
Before this commit: robot URDF, 81 links, 80 joints
Joints:
- joint Head_Roll: limit lower=-0.5235987755982988 upper=0.5235987755982988 effort=6.0 velocity=45.0 -> lower=-0.25 upper=0.25 effort=6.0 velocity=45.0
